File: wordclock.sch (KiCad schematic (older format))
At the start: 24 parts, among them CON1 AVR-ISP-6, J1 UART, J2 Jack-DC, J3 Screw_Terminal_01x03, SW1 SW_Push, SW2 SW_Push, U1 ATMEGA168PA-PU, U2 DS1307+, Y1 16MHz, Y2 32.7680kHz

Commit message: added ignore file
Parts:
- IC1: renamed from U1; symbol ATMEGA168PA-PU -> ATMEGA168PA-PU-RESCUE-wordclock
- J1: value UART -> UAR7
- J3: value Screw_Terminal_01x03 -> Neo Pixel
- Y2: footprint Crystals:Crystal_C38-LF_d3.0mm_l8.0mm_Horizontal -> Crystals:Crystal_C18-LF_d3.0mm_l8.0mm_Horizontal
- renumbered C3 to C1, C1 to C3, U2 to IC2, R3 to R1, R7 to R2, R6 to R5, R5 to R6, R1 to R7, R2 to R8
Connections:
- net +5V: now also C3.1; no longer C5.1
- net at IC1.21 (AREF): now also C5.1; no longer C3.1
- net RTS renamed R7S
Other:
- moved on the sheet: C3, C4, C5
Changed lines of the file:
@@
 EESchema Schematic File Version 2
+LIBS:wordclock-rescue
 LIBS:power
 LIBS:device
@@
 $EndDescr
 $Comp
-L R R3
+L R R1
 U 1 1 5A1AE280
 P 4050 6350
-F 0 "R3" V 4130 6350 50  0000 C CNN
+F 0 "R1" V 4130 6350 50  0000 C CNN
 F 1 "10k" V 4050 6350 50  0000 C CNN
 F 2 "Resistors_THT:R_Axial_DIN0204_L3.6mm_D1.6mm_P7.62mm_Horizontal" V 3980 6350 50  0001 C CNN
@@
 P 4050 4300
 F 0 "J3" H 4050 4500 50  0000 C CNN
-F 1 "Screw_Terminal_01x03" H 4050 4100 50  0000 C CNN
+F 1 "Neo Pixel" H 4050 4100 50  0000 C CNN
 F 2 "Connectors_Terminal_Blocks:TerminalBlock_Philmore_TB133_03x5mm_Straight" H 4050 4300 50  0001 C CNN
 F 3 "" H 4050 4300 50  0001 C CNN
@@
 TX
 Text Label 1050 3800 2    60   ~ 0
-RTS
+R7S
 $Comp
 L Conn_01x04_Male J1
@@
 P 700 4000
 F 0 "J1" H 700 4200 50  0000 C CNN
-F 1 "UART" H 700 3700 50  0000 C CNN
+F 1 "UAR7" H 700 3700 50  0000 C CNN
 F 2 "Pin_Headers:Pin_Header_Straight_1x04_Pitch2.54mm" H 700 4000 50  0001 C CNN
 F 3 "" H 700 4000 50  0001 C CNN
@@
 	4700 6700 4600 6800
 Text Label 4600 6550 2    60   ~ 0
-RTS
+R7S
 Text Label 4600 6700 2    60   ~ 0
 RX
@@
 $EndComp
 $Comp
-L R R7
+L R R2
 U 1 1 5A1B0D5B
 P 5750 5950
-F 0 "R7" V 5830 5950 50  0000 C CNN
+F 0 "R2" V 5830 5950 50  0000 C CNN
 F 1 "10k" V 5750 5950 50  0000 C CNN
 F 2 "Resistors_THT:R_Axial_DIN0204_L3.6mm_D1.6mm_P7.62mm_Horizontal" V 5680 5950 50  0001 C CNN
@@
 $EndComp
 $Comp
-L DS1307+ U2
+L DS1307+ IC2
 U 1 1 5A1B0F47
 P 1850 2650
-F 0 "U2" H 2120 3200 50  0000 C CNN
+F 0 "IC2" H 2120 3200 50  0000 C CNN
 F 1 "DS1307+" H 2150 2100 50  0000 C CNN
 F 2 "Housings_DIP:DIP-8_W7.62mm_Socket_LongPads" H 1850 2650 50  0001 C CNN
@@
 F 0 "Y2" H 1050 3100 50  0000 C CNN
 F 1 "32.7680kHz" H 1050 2800 50  0000 C CNN
-F 2 "Crystals:Crystal_C38-LF_d3.0mm_l8.0mm_Horizontal" H 1050 2950 50  0001 C CNN
+F 2 "Crystals:Crystal_C18-LF_d3.0mm_l8.0mm_Horizontal" H 1050 2950 50  0001 C CNN
 F 3 "" H 1050 2950 50  0001 C CNN
 	1    1050 2950
@@
 NoConn ~ 2450 2350
 $Comp
-L R R6
+L R R5
 U 1 1 5A1B1AAD
 P 1200 2150
-F 0 "R6" V 1280 2150 50  0000 C CNN
+F 0 "R5" V 1280 2150 50  0000 C CNN
 F 1 "4.7k" V 1200 2150 50  0000 C CNN
 F 2 "Resistors_THT:R_Axial_DIN0204_L3.6mm_D1.6mm_P7.62mm_Horizontal" V 1130 2150 50  0001 C CNN
@@
 Real Time Clock
 $Comp
-L CP C3
+L CP C1
 U 1 1 5A1B24C9
 P 2900 4300
-F 0 "C3" H 2925 4400 50  0000 L CNN
+F 0 "C1" H 2925 4400 50  0000 L CNN
 F 1 "470uF" H 2925 4200 50  0000 L CNN
 F 2 "Capacitors_THT:CP_Radial_D6.3mm_P2.50mm" H 2938 4150 50  0001 C CNN
@@
 $EndComp
 $Comp
-L R R5
+L R R6
 U 1 1 5A1B2A1B
 P 3650 4300
-F 0 "R5" V 3730 4300 50  0000 C CNN
+F 0 "R6" V 3730 4300 50  0000 C CNN
 F 1 "330R" V 3650 4300 50  0000 C CNN
 F 2 "Resistors_THT:R_Axial_DIN0204_L3.6mm_D1.6mm_P7.62mm_Horizontal" V 3580 4300 50  0001 C CNN
@@
 $EndComp
 $Comp
-L R R2
+L R R8
 U 1 1 5A1B41D2
 P 5600 7200
-F 0 "R2" V 5680 7200 50  0000 C CNN
+F 0 "R8" V 5680 7200 50  0000 C CNN
 F 1 "10k" V 5600 7200 50  0000 C CNN
 F 2 "Resistors_THT:R_Axial_DIN0204_L3.6mm_D1.6mm_P7.62mm_Horizontal" V 5530 7200 50  0001 C CNN
@@
 $EndComp
 $Comp
-L R R1
+L R R7
 U 1 1 5A1B43D0
 P 5350 7200
-F 0 "R1" V 5430 7200 50  0000 C CNN
+F 0 "R7" V 5430 7200 50  0000 C CNN
 F 1 "10k" V 5350 7200 50  0000 C CNN
 F 2 "Resistors_THT:R_Axial_DIN0204_L3.6mm_D1.6mm_P7.62mm_Horizontal" V 5280 7200 50  0001 C CNN
@@
 Power
 $Comp
-L ATMEGA168PA-PU U1
+L ATMEGA168PA-PU-RESCUE-wordclock IC1
 U 1 1 5A1AE21E
 P 2500 6200
-F 0 "U1" H 1750 7450 50  0000 L BNN
+F 0 "IC1" H 1750 7450 50  0000 L BNN
 F 1 "ATMEGA168PA-PU" H 2900 4800 50  0000 L BNN
 F 2 "Housings_DIP:DIP-28_W7.62mm_Socket_LongPads" H 2500 6200 50  0001 C CIN
@@
 I2C
 $Comp
-L C C1
+L C C3
 U 1 1 5A1B87EF
-P 1550 5900
-F 0 "C1" H 1575 6000 50  0000 L CNN
-F 1 "100n" H 1575 5800 50  0000 L CNN
-F 2 "Capacitors_THT:C_Disc_D3.0mm_W1.6mm_P2.50mm" H 1588 5750 50  0001 C CNN
-F 3 "" H 1550 5900 50  0001 C CNN
-	1    1550 5900
+P 1050 5900
+F 0 "C3" H 1075 6000 50  0000 L CNN
+F 1 "100n" H 1075 5800 50  0000 L CNN
+F 2 "Capacitors_THT:C_Disc_D3.0mm_W1.6mm_P2.50mm" H 1088 5750 50  0001 C CNN
+F 3 "" H 1050 5900 50  0001 C CNN
+	1    1050 5900
 	-1   0    0    -1
 $EndComp
@@
 L C C5
 U 1 1 5A1BE5E2
+P 1550 5900
+F 0 "C5" H 1575 6000 50  0000 L CNN
+F 1 "100n" H 1575 5800 50  0000 L CNN
+F 2 "Capacitors_THT:C_Disc_D3.0mm_W1.6mm_P2.50mm" H 1588 5750 50  0001 C CNN
+F 3 "" H 1550 5900 50  0001 C CNN
+	1    1550 5900
+	-1   0    0    -1
+$EndComp
+$Comp
+L C C4
+U 1 1 5A1BE69F
 P 1300 5900
-F 0 "C5" H 1325 6000 50  0000 L CNN
+F 0 "C4" H 1325 6000 50  0000 L CNN
 F 1 "100n" H 1325 5800 50  0000 L CNN
 F 2 "Capacitors_THT:C_Disc_D3.0mm_W1.6mm_P2.50mm" H 1338 5750 50  0001 C CNN
@@
 	-1   0    0    -1
 $EndComp
-$Comp
-L C C4
-U 1 1 5A1BE69F
-P 1050 5900
-F 0 "C4" H 1075 6000 50  0000 L CNN
-F 1 "100n" H 1075 5800 50  0000 L CNN
-F 2 "Capacitors_THT:C_Disc_D3.0mm_W1.6mm_P2.50mm" H 1088 5750 50  0001 C CNN
-F 3 "" H 1050 5900 50  0001 C CNN
-	1    1050 5900
-	-1   0    0    -1
-$EndComp

Commit message: cheanges in wordclock pcb files
Connections:
- net +5V: now also J2.1; no longer J2.2, J2.3
- net GND: now also J2.2, J2.3; no longer J2.1
Changed lines of the file:
@@
 EESchema Schematic File Version 2
-LIBS:wordclock-rescue
 LIBS:power
 LIBS:device
@@
 F 3 "" H 5250 5810 50  0001 C CNN
 	1    5200 5850
-	1    0    0    1
+	1    0    0    -1
 $EndComp
 Text Label 1050 3900 2    60   ~ 0
@@
 	5550 5850 5500 5850
 Wire Wire Line
-	5550 5700 5550 5850
-Wire Wire Line
 	5500 5750 5600 5750
 Connection ~ 5550 5750
@@
 	5500 5950 5600 5950
 Wire Wire Line
-	5550 5950 5550 6000
+	5550 5850 5550 6000
 Connection ~ 5550 5950
 Wire Wire Line
@@
 Wire Wire Line
 	3800 4300 3850 4300
+Wire Wire Line
+	5550 5750 5550 5700
 $EndSCHEMATC
